Commit message: gazebo stuff

File: ros2_ws/src/robot_car_pkg/description/robot_core.xacro (robot description, xacro)
@@ -41,4 +41,7 @@
         </xacro:inertial_box>
     </link>
+    <gazebo reference="chassis">
+        <material>Gazebo/White</material>
+    </gazebo>
     <!-- LEFT BACK WHEEL LINK -->
     <joint name="left_back_wheel_joint" type="continuous">
@@ -64,4 +67,7 @@
         </xacro:inertial_cylinder>
     </link>
+    <gazebo reference="left_back_wheel">
+        <material>Gazebo/Blue</material>
+    </gazebo>
     <!-- LEFT FRONT WHEEL LINK -->
     <joint name="left_front_wheel_joint" type="continuous">
@@ -87,4 +93,7 @@
         </xacro:inertial_cylinder>
     </link>
+    <gazebo reference="left_front_wheel">
+        <material>Gazebo/Blue</material>
+    </gazebo>
     <!-- RIGHT BACK WHEEL LINK -->
     <joint name="right_back_wheel_joint" type="continuous">
@@ -110,4 +119,7 @@
         </xacro:inertial_cylinder>
     </link>
+    <gazebo reference="right_back_wheel">
+        <material>Gazebo/Blue</material>
+    </gazebo>
     <!-- RIGHT BACK WHEEL LINK -->
     <joint name="right_front_wheel_joint" type="continuous">
@@ -133,3 +145,6 @@
         </xacro:inertial_cylinder>
     </link>
+    <gazebo reference="right_front_wheel">
+        <material>Gazebo/Blue</material>
+    </gazebo>
 </robot>

Commit message: Sync

File: ros2_ws/src/robot_car_pkg/description/robot_core.xacro (robot description, xacro)
@@ -3,5 +3,5 @@
     <xacro:include filename="inertial_macros.xacro"/>
     <material name="white">
-        <color rgba="1 1 1 1" />
+        <color rgba="1 1 1 1"/>
     </material>
     <material name="orange">
@@ -16,4 +16,11 @@
     <!-- BASE LINK -->
     <link name="base_link">
+    </link>
+    <joint name="base_footprint_joint" type="fixed">
+        <parent link="base_link"/>
+        <child link="base_footprint"/>
+        <origin xyz="0 0 0" rpy="0 0 0"/>
+    </joint>
+    <link name="base_footprint">
     </link>
     <!-- CHASSIS LINK -->
@@ -74,5 +81,5 @@
         <parent link="base_link"/>
         <child link="left_front_wheel"/>
-        <origin xyz="0.1 0.095 0.0" rpy="-${pi/2} 0 0" />
+        <origin xyz="0.1 0.095 0.0" rpy="-${pi/2} 0 0"/>
         <axis xyz="0 0 1"/>
     </joint>
@@ -100,5 +107,5 @@
         <parent link="base_link"/>
         <child link="right_back_wheel"/>
-        <origin xyz="-0.1 -0.095 0.0" rpy="${pi/2} 0 0" />
+        <origin xyz="-0.1 -0.095 0.0" rpy="${pi/2} 0 0"/>
         <axis xyz="0 0 -1"/>
     </joint>
@@ -126,5 +133,5 @@
         <parent link="base_link"/>
         <child link="right_front_wheel"/>
-        <origin xyz="0.1 -0.095 0.0" rpy="${pi/2} 0 0" />
+        <origin xyz="0.1 -0.095 0.0" rpy="${pi/2} 0 0"/>
         <axis xyz="0 0 -1"/>
     </joint>
