Commit message: sync

File: ros2_ws/install/robot_car_pkg/share/robot_car_pkg/description/robot_core.xacro (robot description, xacro)
@@ -42,5 +42,5 @@
     </link>
     <!-- LEFT BACK WHEEL LINK -->
-    <joint name="left_back_wheel_joint" type="fixed">
+    <joint name="left_back_wheel_joint" type="continuous">
         <parent link="base_link"/>
         <child link="left_back_wheel"/>
@@ -65,5 +65,5 @@
     </link>
     <!-- LEFT FRONT WHEEL LINK -->
-    <joint name="left_front_wheel_joint" type="fixed">
+    <joint name="left_front_wheel_joint" type="continuous">
         <parent link="base_link"/>
         <child link="left_front_wheel"/>
@@ -88,5 +88,5 @@
     </link>
     <!-- RIGHT BACK WHEEL LINK -->
-    <joint name="right_back_wheel_joint" type="fixed">
+    <joint name="right_back_wheel_joint" type="continuous">
         <parent link="base_link"/>
         <child link="right_back_wheel"/>
@@ -111,5 +111,5 @@
     </link>
     <!-- RIGHT BACK WHEEL LINK -->
-    <joint name="right_front_wheel_joint" type="fixed">
+    <joint name="right_front_wheel_joint" type="continuous">
         <parent link="base_link"/>
         <child link="right_front_wheel"/>

File: ros2_ws/src/robot_car_pkg/description/robot_core.xacro (robot description, xacro)
@@ -15,8 +15,4 @@
     </material>
     <!-- BASE LINK -->
-    <joint name="world_to_base", type="floating">
-        <parent link="world"/>
-        <child link="base_link"/>
-    <joint>
     <link name="base_link">
     </link>
@@ -46,5 +42,5 @@
     </link>
     <!-- LEFT BACK WHEEL LINK -->
-    <joint name="left_back_wheel_joint" type="fixed">
+    <joint name="left_back_wheel_joint" type="continuous">
         <parent link="base_link"/>
         <child link="left_back_wheel"/>
@@ -69,5 +65,5 @@
     </link>
     <!-- LEFT FRONT WHEEL LINK -->
-    <joint name="left_front_wheel_joint" type="fixed">
+    <joint name="left_front_wheel_joint" type="continuous">
         <parent link="base_link"/>
         <child link="left_front_wheel"/>
@@ -92,5 +88,5 @@
     </link>
     <!-- RIGHT BACK WHEEL LINK -->
-    <joint name="right_back_wheel_joint" type="fixed">
+    <joint name="right_back_wheel_joint" type="continuous">
         <parent link="base_link"/>
         <child link="right_back_wheel"/>
@@ -115,5 +111,5 @@
     </link>
     <!-- RIGHT BACK WHEEL LINK -->
-    <joint name="right_front_wheel_joint" type="fixed">
+    <joint name="right_front_wheel_joint" type="continuous">
         <parent link="base_link"/>
         <child link="right_front_wheel"/>

Commit message: checkpoint

File: ros2_ws/install/robot_car_pkg/share/robot_car_pkg/description/robot_core.xacro (robot description, xacro)
@@ -3,5 +3,5 @@
     <xacro:include filename="inertial_macros.xacro"/>
     <material name="white">
-        <color rgba="1 1 1 1" />
+        <color rgba="1 1 1 1"/>
     </material>
     <material name="orange">
@@ -16,4 +16,11 @@
     <!-- BASE LINK -->
     <link name="base_link">
+    </link>
+    <joint name="base_footprint_joint" type="fixed">
+        <parent link="base_link"/>
+        <child link="base_footprint"/>
+        <origin xyz="0 0 0" rpy="0 0 0"/>
+    </joint>
+    <link name="base_footprint">
     </link>
     <!-- CHASSIS LINK -->
@@ -41,4 +48,7 @@
         </xacro:inertial_box>
     </link>
+    <gazebo reference="chassis">
+        <material>Gazebo/White</material>
+    </gazebo>
     <!-- LEFT BACK WHEEL LINK -->
     <joint name="left_back_wheel_joint" type="continuous">
@@ -64,9 +74,12 @@
         </xacro:inertial_cylinder>
     </link>
+    <gazebo reference="left_back_wheel">
+        <material>Gazebo/Blue</material>
+    </gazebo>
     <!-- LEFT FRONT WHEEL LINK -->
     <joint name="left_front_wheel_joint" type="continuous">
         <parent link="base_link"/>
         <child link="left_front_wheel"/>
-        <origin xyz="0.1 0.095 0.0" rpy="-${pi/2} 0 0" />
+        <origin xyz="0.1 0.095 0.0" rpy="-${pi/2} 0 0"/>
         <axis xyz="0 0 1"/>
     </joint>
@@ -87,9 +100,12 @@
         </xacro:inertial_cylinder>
     </link>
+    <gazebo reference="left_front_wheel">
+        <material>Gazebo/Blue</material>
+    </gazebo>
     <!-- RIGHT BACK WHEEL LINK -->
     <joint name="right_back_wheel_joint" type="continuous">
         <parent link="base_link"/>
         <child link="right_back_wheel"/>
-        <origin xyz="-0.1 -0.095 0.0" rpy="${pi/2} 0 0" />
+        <origin xyz="-0.1 -0.095 0.0" rpy="${pi/2} 0 0"/>
         <axis xyz="0 0 -1"/>
     </joint>
@@ -110,9 +126,12 @@
         </xacro:inertial_cylinder>
     </link>
+    <gazebo reference="right_back_wheel">
+        <material>Gazebo/Blue</material>
+    </gazebo>
     <!-- RIGHT BACK WHEEL LINK -->
     <joint name="right_front_wheel_joint" type="continuous">
         <parent link="base_link"/>
         <child link="right_front_wheel"/>
-        <origin xyz="0.1 -0.095 0.0" rpy="${pi/2} 0 0" />
+        <origin xyz="0.1 -0.095 0.0" rpy="${pi/2} 0 0"/>
         <axis xyz="0 0 -1"/>
     </joint>
@@ -133,3 +152,6 @@
         </xacro:inertial_cylinder>
     </link>
+    <gazebo reference="right_front_wheel">
+        <material>Gazebo/Blue</material>
+    </gazebo>
 </robot>
