Commit message: controlled the bot in gazebo

File: ros2_ws/install/robot_car_pkg/share/robot_car_pkg/description/robot.urdf.xacro (robot description, xacro)
@@ -2,3 +2,4 @@
 <robot xmlns:xacro="http://www.ros.org/wiki/xacro"  name="robot">
     <xacro:include filename="robot_core.xacro" />
-</robot>l
+    <xacro:include filename="gazebo_control.xacro" />
+</robot>

File: ros2_ws/install/robot_car_pkg/share/robot_car_pkg/description/robot_core.xacro (robot description, xacro)
@@ -16,11 +16,4 @@
     <!-- BASE LINK -->
     <link name="base_link">
-    </link>
-    <joint name="base_footprint_joint" type="fixed">
-        <parent link="base_link"/>
-        <child link="base_footprint"/>
-        <origin xyz="0 0 0" rpy="0 0 0"/>
-    </joint>
-    <link name="base_footprint">
     </link>
     <!-- CHASSIS LINK -->
@@ -78,5 +71,5 @@
     </gazebo>
     <!-- LEFT FRONT WHEEL LINK -->
-    <joint name="left_front_wheel_joint" type="continuous">
+    <joint name="left_front_wheel_joint" type="fixed">
         <parent link="base_link"/>
         <child link="left_front_wheel"/>
@@ -129,6 +122,6 @@
         <material>Gazebo/Blue</material>
     </gazebo>
-    <!-- RIGHT BACK WHEEL LINK -->
-    <joint name="right_front_wheel_joint" type="continuous">
+    <!-- RIGHT FRONT WHEEL LINK -->
+    <joint name="right_front_wheel_joint" type="fixed">
         <parent link="base_link"/>
         <child link="right_front_wheel"/>
